File: Integration/Hardware/Rover/roverPCB.sch (EAGLE design)
At the start: 37 parts, among them IC2 DS3231/SO, IC3 741G53DCT

Commit message: Organized and labeled schematic
Parts:
- removed U$1: MAX3243, ftdi4:MAX3243
- added RF_CONVERT: MAX3243, ftdi4:MAX3243
Connections:
- net 10: now also RF_CONVERT.ROUT2; no longer U$1.ROUT2
- net 3.3V_M0: now also RF_CONVERT.FORCEON, RF_CONVERT.VCC; no longer U$1.FORCEON, U$1.VCC
- net C1+: now also RF_CONVERT.C1+; no longer U$1.C1+
- net FORCEOFF_MAX: now also RF_CONVERT.FORCEOFF_N; no longer U$1.FORCEOFF_N
- net GND: now also RF_CONVERT.DIN2, RF_CONVERT.DIN3, RF_CONVERT.GND; no longer U$1.DIN2, U$1.DIN3, U$1.GND
- net N$10: now also RF_CONVERT.V-; no longer U$1.V-
- net N$11: now also RF_CONVERT.C1-; no longer U$1.C1-
- net N$13: now also RF_CONVERT.V+; no longer U$1.V+
- net N$4: now also RF_CONVERT.C2+; no longer U$1.C2+
- net N$5: now also RF_CONVERT.C2-; no longer U$1.C2-
- net RS232_CD_FROM_RADIO: now also RF_CONVERT.RIN2; no longer U$1.RIN2
- net RS232_TX_FROM_M0: now also RF_CONVERT.DOUT1; no longer U$1.DOUT1
- net RS232_TX_FROM_RADIO: now also RF_CONVERT.RIN1; no longer U$1.RIN1
- net TX: now also RF_CONVERT.DIN1; no longer U$1.DIN1
- net TX_FROM_RADIO: now also RF_CONVERT.ROUT1; no longer U$1.ROUT1
Other:
- note added: "Data logging and RTC"
- note added: "Debug and jumper pins"
- note added: "Microcontroller and Accelerometer"
- note added: "Power Circuitry"
- note added: "Radio and Telemetry ICs"
- note added: "Relay Control"
- note removed: "A2, A4, 13, 9"
- note removed: "FIXES!! DIN -- > GND IF USING TTL ACCELEROMETER MOUNTED TO BOARD RADIO INTERUPT PIN PASSIVELY HIGH COVER VIAS WITH SOLDER MASK PLACE ALL IC'S ON 3.3V FROM FEATHER"
- note removed: "Included this particular RS232 driver in case we ever have a need to tap into the diagnostic ports of the Z9-C"
- note removed: "Look into attaching the low side driver to the inhibitable VCC"
- note removed: "expose all free pins on the 4 header connector"
- note removed: "optionally tie 13 to enable of second rail"
- note removed: "verify that this chip can run on siad voltage"
- moved on the sheet: C1, C2, C3, C4, C5, C6, C7, CBYPASS, IC2, IC3, J1, J4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
