File: Integration/Hardware/Base/BasePCB.sch (EAGLE design)
At the start: 33 parts, among them IC3 741G53DCT

Commit message: Organized schematic
Other:
- note added: "Microcontroller and datalogging"
- note added: "Periphreal Interfaces"
- note added: "Power Circuitry"
- note added: "Radio Telemetry Circuitry"
- note added: "Relay Circuitry"
- note removed: "JUMPERS VERIFIED"
- moved on the sheet: C1, C2, C3, C4, C5, CBYPASS, EN_VCC2, GNSS_PWR, IC3, J1, J2, J4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
